File: hw-charger.kicad_pcb (KiCad board)
At the start: 4 copper layers, 100 x 65 mm, 164 parts, among them J10 Screw_Terminal_01x02, J17 Conn_01x02, J19 Conn_01x02, J2 Conn_02x04_Odd_Even, J27 Conn_01x05, J3 Screw_Terminal_01x03, J4 Conn_02x05_Odd_Even, J56 Screw_Terminal_01x02, J57 Conn_01x02, J58 Screw_Terminal_01x02, J59 Conn_01x02, J60 Screw_Terminal_01x02, J61 Conn_01x02, J62 Screw_Terminal_01x02, J63 Conn_01x02, J9 Conn_01x02, Q6 BSC0702LS, Q7 BSC0702LS, Q8 BSC0702LS, Q9 BSC0702LS, U1 ME6203A50M3G, U14 Fuse Holder, U15 Fuse Holder, U16 Fuse Holder, U17 Fuse Holder, U2 Jumper Black, U27 BQ25756RRVR, U3 Jumper Black, U72 Jumper Red, U73 Jumper Blue, U74 Fuse 2A, U75 Fuse 2A

Commit message: Fixed CE pin connection; Use git version as variable
Parts:
- moved R21 2.00 mm to (63.9, 195.8)
- moved R75 2.00 mm to (63.9, 193.8), turned to 90 degrees
Connections:
- R75 pad 1: Net-(TP3-A) -> Net-(TP3-C)
- TP3 pad 1: Net-(TP3-A) -> unconnected-(TP3-A-Pad1)
Routing:
- net Net-(TP3-A): track 2.60 -> 0.00 mm
- net Net-(TP3-C): track 55.0 -> 57.4 mm
- net GND: track 35.5 -> 36.5 mm, vias 138 -> 139
- net /V_CHARGE: track 166.2 -> 167.0 mm
Other:
- board text added: "Charger ${git_version} License CC BY 4.0 github.com/xtech/hw-charger"
- board text removed: "Charger v0.1.0 License CC BY 4.0 github.com/xtech/hw-charger"
